File: pcb/kalmar.kicad_pcb (KiCad board)
At the start: 2 copper layers, 129.9 x 95.6 mm, 27 parts, among them J1 MJ-4PP-9, SW1 SW_SPDT

Commit message: v0.3
fix connection
add jack cut
Parts:
- added ?: , , F.Cu at (185.2, 78.6)
- added ?: , , F.Cu at (184.0, 92.2)
- J1: footprint enki_lib:MJ-4PP-9_dual -> enki_lib:MJ-4PP-9_dual_topor
- SW1: footprint enki_lib:switch_MSK-12C02_smd_x2 -> enki_lib:switch_MSK-12C02_smd_x2_topor
- moved H1 103.8 mm to (163.4, 120.1)
- moved H2 103.8 mm to (145.1, 87.2)
- moved H3 103.8 mm to (84.2, 79.9)
- moved H5 103.8 mm to (90.6, 107.9)
- moved SW1 103.8 mm to (179.6, 118.0)
- moved SWr1c3 103.8 mm to (116.5, 55.2)
- moved SWr2c1 103.8 mm to (154.9, 82.4)
- moved SWr2c2 103.8 mm to (137.2, 78.0)
- moved SWr2c3 103.8 mm to (116.5, 72.2)
- moved SWr2c4 103.8 mm to (95.9, 79.6)
- moved SWr2c5 103.8 mm to (77.1, 101.7)
- moved SWr3c3 103.8 mm to (116.5, 89.2)
- moved SWr4c2 103.8 mm to (151.4, 123.3)
- moved G*** 103.8 mm to (119.8, 112.0)
- moved J1 103.8 mm to (187.6, 79.0)
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- renumbered U to U1
Connections:
- SWr3c5 pad : r3c5 -> (no net)
- U1 pad 16: r3c3 -> r3c2
Routing:
- net r3c3: track 145.4 -> 94.3 mm, vias 2 -> 1
- net reset: track 83.1 -> 38.5 mm, vias 3 -> 2
- net r3c2: track 30.0 -> 71.8 mm, vias 0 -> 1
- net r3c5: track 181.7 -> 140.4 mm
- net r4c2: track 99.5 -> 61.5 mm, vias 0 -> 1
- net r2c3: track 136.6 -> 98.6 mm
- net r1c5: track 179.2 -> 145.4 mm, vias 2 -> 1
- net r2c1: track 72.4 -> 49.8 mm, vias 1 -> 2
- net VBAT: track 74.7 -> 53.5 mm, vias 4 -> 2
- net data: track 48.6 -> 27.6 mm, vias 2 -> 1
- net r2c4: track 144.9 -> 126.8 mm
- net r2c5: track 148.3 -> 130.9 mm, vias 2 -> 1
- net r1c1: track 72.5 -> 87.8 mm
- net GND: track 751.3 -> 739.3 mm
- net r3c4: track 131.0 -> 119.8 mm
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Other:
- outline, holes or cut-outs redrawn
- board text added: "original by tapioki modded by Aroum"
- board text removed: "original by tapioki modded by Aroum v0.2"
